Commit message: update efforts

File: sim/resources/gpr/robot_fixed.urdf (robot description, URDF)
Before this commit: robot gpr, 22 links, 21 joints
Joints:
- joint L_ankle_y: limit lower=-0.6981317 upper=0.6981317 effort=50 velocity=10 -> lower=-0.6981317 upper=0.6981317 effort=17 velocity=10
- joint L_hip_x: limit lower=-0.34906585 upper=3.1852259 effort=100 velocity=10 -> lower=-0.34906585 upper=3.1852259 effort=60 velocity=10
- joint L_hip_z: limit lower=-1.5707963 upper=1.5707963 effort=100 velocity=10 -> lower=-1.5707963 upper=1.5707963 effort=60 velocity=10
- joint R_ankle_y: limit lower=-0.6981317 upper=0.6981317 effort=50 velocity=10 -> lower=-0.6981317 upper=0.6981317 effort=17 velocity=10
- joint R_hip_x: limit lower=-0.34906585 upper=3.1852259 effort=100 velocity=10 -> lower=-0.34906585 upper=3.1852259 effort=60 velocity=10
- joint R_hip_z: limit lower=-1.5707963 upper=1.5707963 effort=100 velocity=10 -> lower=-1.5707963 upper=1.5707963 effort=60 velocity=10
